File: Eagle_file/pcb.sch (EAGLE design)
At the start: 19 parts, among them IC1 BL8555-33, K1 usb_probe, Q1 BSS123, Q2 BSS123, T1 BC547, T2 BC547

Commit message: Update pcb board
Parts:
- removed K1: usb_probe, Wuerth_Elektronik_eiCan_Communication_Connectors_v2.2:629105136821
- added IC2: LM358N, linear:LM358N
- added JP2: Step Up, pinhead:PINHD-1X4
- added R10, R8: 100k, rcl:R-EU_0204/7
- added R11, R9: 1M, rcl:R-EU_0204/7
- added R7: 1K, rcl:R-EU_0204/7
- added SV1: MPX2050, con-lstb:MA04-1
- added USB1: MOLEX-47346-0001, usb_con-update:MOLEX-47346-0001
- R5: value 1K -> 250
- U$1: value (none) -> stm32f103c8t6
Connections:
- new net 10V: JP2.2, SV1.3
- new net 3.3VS: C2.2, C3.2, IC1.OUT, USB1.1
- new net N$10: IC2A.+IN, R10.2, R11.2
- new net N$7: Q2.D, R2.1, USB1.2
- new net N$9: IC2A.-IN, R8.2, R9.1
- new net PA0: IC2A.OUT, R9.2, U$1.PA0
- new net V+: R8.1, SV1.2
- new net V-: R10.1, SV1.4
- net 3.3V: now also IC2P.V+, U$1.3.3V1; no longer C2.2, C3.2, IC1.OUT, K1.1, K1.2, Q2.D, R2.1
- net GND: now also IC2P.V-, JP2.3, JP2.4, R11.1, SV1.1, USB1.5, USB1.GND1, USB1.GND2, USB1.GND3, USB1.GND4; no longer K1.5
- net LED: now also R5.2, USB1.3; no longer K1.3
- net N$4: now also R7.2; no longer R6.2
- net N$6: now also R6.2; no longer R5.2
- net PB6: now also R6.1; no longer R5.1
- net PB7: now also R7.1; no longer R6.1
- net PB8: now also Q2.S, R1.1; no longer Q1.S, R3.1
- net PB9: now also Q1.S, R3.1; no longer Q2.S, R1.1
- net SDA: now also USB1.4; no longer K1.4
- net VCC: now also JP2.1, R5.1
Other:
- note added: "Blue Pill"
- note added: "Control modul"
- note added: "MPX2050"
- moved on the sheet: D1, D2, JP1, R5, R6, T1, T2
